File: Transplutonic-Resonator.kicad_sch (KiCad schematic)
At the start: 10 parts, among them U1 LT8491EUKJ-PBF

Commit message: Added voltage sensor, dc/solar detector, V_IN Partially added battery voltage limiter (stage 2 charge max batt charge voltage)
Parts:
- removed C1: 8.2nF, symbol Device:C
- removed C2: 220pF, symbol Device:C
- removed C3: 68nF, symbol Device:C
- removed D1: LED, symbol Device:LED
- removed R1: 10kohm, symbol Device:R
- removed R2: 53.6kohm, symbol Device:R
- removed R3: 1.3kohm, symbol Device:R
- removed R4: 100kohm, symbol Device:R
- removed R5: 549ohm, symbol Device:R
Connections:
- net GND: no longer U1.21 (SYNC)
- net Input Voltage Sensor/FBIR_out: now reaches U1.1 (FBIR)
- net Input Voltage Sensor/FBIN_out: now reaches U1.15 (FBIN)
- net VINR Resistor Divider/VINR_out: now reaches U1.54 (VINR)
- net Input Voltage Sensor/FBIW_out: now reaches U1.6 (FBIW)
Other:
- added sheet Battery Voltage Limiter (batt_v_limiter.kicad_sch)
- added sheet Input Voltage Sensor (input_voltage_sensor.kicad_sch)
- added sheet VINR Resistor Divider (vinr_resistor_divider.kicad_sch)
- company: (none) -> Az Builds
- title: (none) -> Transplutonic Resonator
